File: MiniCopterSchematic/MiniCopterSchematic.kicad_sch (KiCad schematic)
At the start: 11 parts

Commit message: Working on schematic
Parts:
- removed U?: MPU-6050, Sensor_Motion:InvenSense_QFN-24_4x4mm_P0.5mm, symbol Sensor_Motion:MPU-6050
- added A?: Arduino_UNO_R3, Module:Arduino_UNO_R3, symbol MCU_Module:Arduino_UNO_R3
- added J? (x2): JOYSTICK_BREAKOUT, symbol AA_Custom_Components:JOYSTICK_BREAKOUT
- added J?: MPU6050_IMU, symbol AA_Custom_Components:MPU6050_IMU
- added U?: NRF24L01_Breakout, RF_Module:nRF24L01_Breakout, symbol RF:NRF24L01_Breakout
Connections:
- net GNDREF is gone; now on net GND: Q?.3 (S), Q?.3 (S), Q?.3 (S), Q?.3 (S)
- net +BATT: now also A?.27 (+5V), U?.2 (VCC), J?.7 (VCC), U?.2 (VCC)
- net CE: now also U?.3 (CE)
- net CSN: now also U?.4 (~{CSN})
- net MISO: now also U?.7 (MISO)
- net MOSI: now also U?.6 (MOSI)
- net SCK: now also U?.5 (SCK)
- net GND: now reaches U?.1 (GND)
- net GND: now also A?.29 (GND), A?.4 (GND), J?.1 (INT), J?.6 (GND), U?.1 (GND)
- net SDA: now reaches A?.23 (SDA/A4)
- net SDA: now also J?.3 (SDA)
- net SCL: now reaches A?.24 (SCL/A5)
- net SCL: now also J?.4 (SCL)
- net INT: now reaches A?.5 (D2)
- net INT: now also J?.1 (INT)
Other:
- moved on the sheet: A?, M?, Q?, U?

Commit message: Updating schematic
Connections:
- net +BATT: now also A?.5 (+5V), J?.~ (VRY), J?.~ (VRY)
- net GND: now also A?.7 (GND), J?.~ (VRY), J?.~ (VRY)
- net JOY2_Y: now reaches J?.~ (VRY)
- net JOY2_Y: now also A?.12 (A3)
- net JOY1_Y: now reaches A?.10 (A1)
- net JOY1_Y: now also J?.~ (VRY)
- net JOY2_X: now reaches A?.11 (A2)
- net JOY2_X: now also J?.~ (VRY)
- net JOY1_X: now reaches A?.9 (A0)
- net JOY1_X: now also J?.~ (VRY)
- net CE renamed CE_NANO
- net CE_NANO: no longer U?.3 (CE)
- net CSN renamed CSN_NANO
- net CSN_NANO: no longer U?.4 (~{CSN})
- net MISO renamed MISO_NANO
- net MISO_NANO: no longer U?.7 (MISO)
- net MOSI renamed MOSI_NANO
- net MOSI_NANO: no longer U?.6 (MOSI)
- net SCK renamed SCK_NANO
- net SCK_NANO: no longer U?.5 (SCK)
- new net CE_UNO: U?.3 (CE)
- new net CSN_UNO: U?.4 (~{CSN})
- new net JOY1_BTN: J?.~ (VRY)
- new net MISO_UNO: U?.7 (MISO)
- new net MOSI_UNO: U?.6 (MOSI)
- new net SCK_UNO: U?.5 (SCK)
Other:
- moved on the sheet: U?

Commit message: Finished Schematic
Parts:
- added R? (x4): 10K Ω, symbol Device:R_Small_US
- A?: value Arduino_Nano_Every -> ARDUINO NANO EVERY
- JOYSTICK_1, JOYSTICK_2: renamed from J?; value JOYSTICK_BREAKOUT -> BREAKOUT
- M? (x4): value Motor_DC -> MOTOR_DC
- NRF24L01: renamed from U?; value NRF24L01_Breakout -> BREAKOUT
- ss: renamed from A?; value Arduino_UNO_R3 -> ARDUINO_UNO
Connections:
- net CE_UNO: now also ss.22 (D7)
- net CSN_UNO: now also ss.23 (D8)
- net GND: now also R?.2, R?.2, R?.2, R?.2
- net JOY1_BTN: now also ss.17 (D2)
- net MISO_UNO: now also ss.27 (D12)
- net MOSI_UNO: now also ss.26 (D11)
- net MOTOR_1: now also R?.1
- net MOTOR_2: now also R?.1
- net MOTOR_3: now also R?.1
- net MOTOR_4: now also R?.1
- net SCK_UNO: now also ss.28 (D13)
- net JOY2_BTN: now reaches ss.18 (D3)
Other:
- note added: "ARDUINO NANO (RECIEVER)"
- note added: "ARDUINO UNO (TRANSMITTER)"
- note added: "MOTORS, MOSFETS"
- note added: "Mini-Copter"
- note added: "ON QUADCOPTER"
- title: (none) -> Mini-Copter
- moved on the sheet: JOYSTICK_1, JOYSTICK_2, NRF24L01

Commit message: Updated schematic
Other:
- note added: "Note: 5V and GND for Transmitter and Reciever are different. All Transmitter parts have same GND and 5V, and all Reciever parts have same GND and 5V."
Changed lines of the file:
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@@
     (effects (font (size 12 12) (thickness 1.4) bold italic) (justify left bottom))
+  )
+  (text "Note: 5V and GND for Transmitter and Reciever are different. All Transmitter\nparts have same GND and 5V, and all Reciever parts have same GND and 5V."
+    (at 193.04 21.59 0)
+    (effects (font (size 1.27 1.27)) (justify left bottom))
   )
   (text "ARDUINO UNO (TRANSMITTER)" (at 181.61 35.56 0)

Commit message: Working on organizing perfboard
Parts:
- removed R? (x2): 10K Ω, symbol Device:R_Small_US
- added R? (x2): 10K Ω, symbol Device:R_Small_US
- gave numbers to parts that had none: 12
- renumbered NRF24L01 to NRF24L01_1, NRF24L01 to NRF24L01_2, ss to ss1
Connections:
- net GND: now also R?.2, R?.2
- net MOTOR_3: now also A1.19 (A0), R?.1; no longer A1.8 (D5)
- net MOTOR_4: now also A1.20 (A1), R?.1; no longer A1.9 (D6)
Other:
- note added: "MINI-COPTER"
- note removed: "Mini-Copter"
- moved on the sheet: R1, R2

Commit message: Updated schematic
Parts:
- gave numbers to parts that had none: 2
Connections:
- net MOTOR_2: now also A1.8 (D5); no longer A1.7 (D4)
- net MOTOR_4: now also A1.21 (A2); no longer A1.20 (A1)
Other:
- moved on the sheet: R2, R4

Commit message: Updated schematic
Connections:
- net MOTOR_3: now also A1.12 (D9); no longer A1.19 (A0)
- net MOTOR_4: now also A1.13 (D10); no longer A1.21 (A2)
Other:
- moved on the sheet: R1, R2, R3, R4

Commit message: Combined MPU and nRF code
Parts:
- M1: value MOTOR_DC -> MOTOR_DC_1
- M2: value MOTOR_DC -> MOTOR_DC_2
- M3: value MOTOR_DC -> MOTOR_DC_3
- M4: value MOTOR_DC -> MOTOR_DC_4
- Q1, Q2, Q3, Q4: value IRF540N -> FQP20NO6L
Changed lines of the file:
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@@
   (title_block
     (title "Mini-Copter")
-    (date "2023-01-28")
+    (date "2023-01-30")
     (rev "1")
     (comment 4 "By: Ashish Agrahari")
@@
     )
   )
-  (global_label "INT" (shape output) (at 62.23 96.52 180) (fields_autoplaced)
+  (global_label "INT" (shape input) (at 62.23 96.52 180) (fields_autoplaced)
     (effects (font (size 1.27 1.27)) (justify right))
     (property "Intersheet References" "${INTERSHEET_REFS}" (id 0) (at 56.914 96.4406 0)
@@
     )
   )
-  (global_label "SDA" (shape output) (at 138.43 128.27 0) (fields_autoplaced)
+  (global_label "SDA" (shape bidirectional) (at 138.43 128.27 0) (fields_autoplaced)
     (effects (font (size 1.27 1.27)) (justify left))
     (property "Intersheet References" "${INTERSHEET_REFS}" (id 0) (at 144.4112 128.1906 0)
@@
     )
   )
-  (global_label "SDA" (shape output) (at 96.52 119.38 0) (fields_autoplaced)
+  (global_label "SDA" (shape bidirectional) (at 96.52 119.38 0) (fields_autoplaced)
     (effects (font (size 1.27 1.27)) (justify left))
     (property "Intersheet References" "${INTERSHEET_REFS}" (id 0) (at 102.5012 119.3006 0)
@@
     )
   )
-  (global_label "SCL" (shape output) (at 138.43 125.73 0) (fields_autoplaced)
+  (global_label "SCL" (shape bidirectional) (at 138.43 125.73 0) (fields_autoplaced)
     (effects (font (size 1.27 1.27)) (justify left))
     (property "Intersheet References" "${INTERSHEET_REFS}" (id 0) (at 144.3507 125.6506 0)
@@
     )
   )
-  (global_label "SCL" (shape output) (at 96.52 121.92 0) (fields_autoplaced)
+  (global_label "SCL" (shape bidirectional) (at 96.52 121.92 0) (fields_autoplaced)
     (effects (font (size 1.27 1.27)) (justify left))
     (property "Intersheet References" "${INTERSHEET_REFS}" (id 0) (at 102.4407 121.8406 0)
@@
   )
   (symbol (lib_id "Transistor_FET:IRF540N") (at 39.37 181.61 0) (unit 1)
-    (in_bom yes) (on_board yes) (fields_autoplaced)
+    (in_bom yes) (on_board yes)
     (property "Reference" "Q1" (id 0) (at 45.72 180.3399 0)
       (effects (font (size 1.27 1.27)) (justify left) hide)
     )
-    (property "Value" "IRF540N" (id 1) (at 45.72 181.6099 0)
+    (property "Value" "FQP20NO6L" (id 1) (at 44.45 184.15 0)
       (effects (font (size 1.27 1.27)) (justify left))
     )
@@
       (effects (font (size 1.27 1.27)) (justify left) hide)
     )
-    (property "Value" "MOTOR_DC" (id 1) (at 92.71 177.8 0)
+    (property "Value" "MOTOR_DC_3" (id 1) (at 91.44 179.07 0)
       (effects (font (size 1.27 1.27)) (justify left))
     )
@@
       (effects (font (size 1.27 1.27)) (justify left) hide)
     )
-    (property "Value" "MOTOR_DC" (id 1) (at 17.78 176.53 0)
+    (property "Value" "MOTOR_DC_1" (id 1) (at 17.78 180.34 0)
       (effects (font (size 1.27 1.27)) (justify left))
     )
@@
       (effects (font (size 1.27 1.27)) (justify left) hide)
     )
-    (property "Value" "MOTOR_DC" (id 1) (at 55.88 177.8 0)
+    (property "Value" "MOTOR_DC_2" (id 1) (at 54.61 179.07 0)
       (effects (font (size 1.27 1.27)) (justify left))
     )
@@
   )
   (symbol (lib_id "Transistor_FET:IRF540N") (at 152.4 181.61 0) (unit 1)
-    (in_bom yes) (on_board yes) (fields_autoplaced)
+    (in_bom yes) (on_board yes)
     (property "Reference" "Q4" (id 0) (at 158.75 180.3399 0)
       (effects (font (size 1.27 1.27)) (justify left) hide)
     )
-    (property "Value" "IRF540N" (id 1) (at 158.75 181.6099 0)
+    (property "Value" "FQP20NO6L" (id 1) (at 157.48 184.15 0)
       (effects (font (size 1.27 1.27)) (justify left))
     )
@@
   )
   (symbol (lib_id "Transistor_FET:IRF540N") (at 77.47 181.61 0) (unit 1)
-    (in_bom yes) (on_board yes) (fields_autoplaced)
+    (in_bom yes) (on_board yes)
     (property "Reference" "Q2" (id 0) (at 83.82 180.3399 0)
       (effects (font (size 1.27 1.27)) (justify left) hide)
     )
-    (property "Value" "IRF540N" (id 1) (at 83.82 181.6099 0)
+    (property "Value" "FQP20NO6L" (id 1) (at 82.55 184.15 0)
       (effects (font (size 1.27 1.27)) (justify left))
     )
@@
       (effects (font (size 1.27 1.27)) (justify left) hide)
     )
-    (property "Value" "MOTOR_DC" (id 1) (at 130.81 177.8 0)
+    (property "Value" "MOTOR_DC_4" (id 1) (at 129.54 179.07 0)
       (effects (font (size 1.27 1.27)) (justify left))
     )
@@
   )
   (symbol (lib_id "Transistor_FET:IRF540N") (at 114.3 181.61 0) (unit 1)
-    (in_bom yes) (on_board yes) (fields_autoplaced)
+    (in_bom yes) (on_board yes)
     (property "Reference" "Q3" (id 0) (at 120.65 180.3399 0)
       (effects (font (size 1.27 1.27)) (justify left) hide)
     )
-    (property "Value" "IRF540N" (id 1) (at 120.65 181.6099 0)
+    (property "Value" "FQP20NO6L" (id 1) (at 119.38 184.15 0)
       (effects (font (size 1.27 1.27)) (justify left))
     )
@@
     )
     (path "/472c65e8-70f2-44ac-9f2a-716990e7abee"
-      (reference "M1") (unit 1) (value "MOTOR_DC") (footprint "")
+      (reference "M1") (unit 1) (value "MOTOR_DC_1") (footprint "")
     )
     (path "/4a8f6f9e-35f2-4e1f-aaa0-443b0c34e52c"
-      (reference "M2") (unit 1) (value "MOTOR_DC") (footprint "")
+      (reference "M2") (unit 1) (value "MOTOR_DC_2") (footprint "")
     )
     (path "/28f52bba-b454-4854-be1d-e6e5fed8c248"
-      (reference "M3") (unit 1) (value "MOTOR_DC") (footprint "")
+      (reference "M3") (unit 1) (value "MOTOR_DC_3") (footprint "")
     )
     (path "/b01074cd-55cf-43fd-b903-6ced15225495"
-      (reference "M4") (unit 1) (value "MOTOR_DC") (footprint "")
+      (reference "M4") (unit 1) (value "MOTOR_DC_4") (footprint "")
     )
     (path "/552c74fa-1e18-46c0-a1b0-07a3fd1d445f"
@@
     )
     (path "/075952fe-8e15-4d5e-bc3f-1b285719d921"
-      (reference "Q1") (unit 1) (value "IRF540N") (footprint "Package_TO_SOT_THT:TO-220-3_Vertical")
+      (reference "Q1") (unit 1) (value "FQP20NO6L") (footprint "Package_TO_SOT_THT:TO-220-3_Vertical")
     )
     (path "/65cbdf8f-c7cf-46fb-bbba-0a529ce80d6c"
-      (reference "Q2") (unit 1) (value "IRF540N") (footprint "Package_TO_SOT_THT:TO-220-3_Vertical")
+      (reference "Q2") (unit 1) (value "FQP20NO6L") (footprint "Package_TO_SOT_THT:TO-220-3_Vertical")
     )
     (path "/b77c14e1-0eba-481e-be9b-8b75dfd5122a"
-      (reference "Q3") (unit 1) (value "IRF540N") (footprint "Package_TO_SOT_THT:TO-220-3_Vertical")
+      (reference "Q3") (unit 1) (value "FQP20NO6L") (footprint "Package_TO_SOT_THT:TO-220-3_Vertical")
     )
     (path "/5003c775-5f69-454f-95ef-75895c4d6035"
-      (reference "Q4") (unit 1) (value "IRF540N") (footprint "Package_TO_SOT_THT:TO-220-3_Vertical")
+      (reference "Q4") (unit 1) (value "FQP20NO6L") (footprint "Package_TO_SOT_THT:TO-220-3_Vertical")
     )
     (path "/c5ef0e82-3e4c-4634-8c5d-728fec12aa1d"
