File: Images/MiniCopterSchematicWithTransmitter/MiniCopterSchematic.kicad_sch (KiCad schematic)
At the start: 17 parts, among them M1 MOTOR_DC_1, M2 MOTOR_DC_2, M3 MOTOR_DC_3, M4 MOTOR_DC_4, Q1 FQP20NO6L, Q2 FQP20NO6L, Q3 FQP20NO6L, Q4 FQP20NO6L

Commit message: Working on PCB for copter
Parts:
- added A2: ARDUINO_UNO, Module:Arduino_UNO_R3, symbol MCU_Module:Arduino_UNO_R3
- added JOYSTICK_1, JOYSTICK_2: BREAKOUT, symbol AA_Custom_Components:JOYSTICK_BREAKOUT
- added NRF24L01_2: BREAKOUT, AA_Custom_Components:NRF24L01_Breakout, symbol RF:NRF24L01_Breakout
Connections:
- net +BATT: now also A2.5 (+5V), JOYSTICK_1.~ (VRY), JOYSTICK_2.~ (VRY), NRF24L01_2.2 (VCC)
- net GND: now also A2.7 (GND), JOYSTICK_1.~ (VRY), JOYSTICK_2.~ (VRY), NRF24L01_2.1 (GND)
- new net CE_UNO: A2.22 (D7), NRF24L01_2.3 (CE)
- new net CSN_UNO: A2.23 (D8), NRF24L01_2.4 (~{CSN})
- new net JOY1_BTN: A2.17 (D2), JOYSTICK_2.~ (VRY)
- new net JOY1_X: A2.9 (A0), JOYSTICK_1.~ (VRY)
- new net JOY1_Y: A2.10 (A1), JOYSTICK_1.~ (VRY)
- new net JOY2_BTN: A2.18 (D3)
- new net JOY2_X: A2.11 (A2), JOYSTICK_2.~ (VRY)
- new net JOY2_Y: A2.12 (A3), JOYSTICK_2.~ (VRY)
- new net MISO_UNO: A2.27 (D12), NRF24L01_2.7 (MISO)
- new net MOSI_UNO: A2.26 (D11), NRF24L01_2.6 (MOSI)
- new net SCK_UNO: A2.28 (D13), NRF24L01_2.5 (SCK)
Other:
- note added: "ARDUINO UNO (TRANSMITTER)"
- note added: "Note: 5V and GND for Transmitter and Reciever are different. All Transmitter parts have same GND and 5V, and all Reciever parts have same GND and 5V."
