File: Images/MiniCopterTransmitterSchematic/MiniCopterTransmitterSchematic.kicad_sch (KiCad schematic)
At the start: 4 parts

Commit message: Finalized PCB
Other:
- note added: "MINI-COPTER JOYSTICK"
- note removed: "(PARTS ON JOYSTICK)"
- note removed: "MINI-COPTER"
Changed lines of the file:
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@@
     (stroke (width 0) (type default) (color 0 0 0 0))
   )
-  (text "(PARTS ON JOYSTICK)" (at 53.34 48.26 0)
-    (effects (font (size 4 4)) (justify left bottom))
-  )
-  (text "MINI-COPTER" (at 26.67 39.37 0)
+  (text "MINI-COPTER JOYSTICK" (at 26.67 39.37 0)
     (effects (font (size 12 12) (thickness 1.4) bold italic) (justify left bottom))
   )

Commit message: Updated schematics and pics
Parts:
- added U2: BUTTON_BREAKOUT, symbol AA_Custom_Components:BUTTON_BREAKOUT
- J1: renamed from JOYSTICK_1; value BREAKOUT -> JOYSTICK_1
- J2: renamed from JOYSTICK_2; value BREAKOUT -> JOYSTICK_2
- U3: renamed from NRF24L01_2; value BREAKOUT -> NRF24L01
- renumbered A2 to U1
Connections:
- net +BATT: now also U2.3 (PIN4)
- net GND: now also U2.4 (PIN3)
- net JOY1_BTN: now also U1.18 (D3); no longer U1.17 (D2)
- net JOY2_BTN: now also U1.19 (D4); no longer U1.18 (D3)
- new net INT_BTN: U1.17 (D2), U2.1 (PIN1)
Other:
- note added: "INTERRUPT BUTTON"
